File: hardware/mfm-v3-smd.kicad_sch (KiCad schematic)
At the start: 47 parts, among them J1 MFM Module-Left, J2 MFM Module-Right, J3 SMBUS Connector, J4 FTDI Connector, J5 ICSP Connector, J6 Antenna, J7 JST Jack, Q1 R.V. Protect, SW1 SW_VBAT, SW2 RESET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

Commit message: fix(hardware): DNP buffer cap
Parts:
- C12: now not fitted
Changed lines of the file:
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@@
   )
   (symbol (lib_id "Device:CP_Small") (at 43.18 27.94 0) (unit 1)
-    (in_bom yes) (on_board yes) (dnp no)
+    (in_bom yes) (on_board yes) (dnp yes)
     (property "Reference" "C12" (at 36.83 27.94 0)
       (effects (font (size 1.27 1.27)) (justify left))
